File: hardware/DSP_Stamp_Mini.kicad_sch (KiCad schematic)
At the start: 73 parts, among them J1 Conn_01x10, J2 SM03B-SRSS-TB, J3 Conn_01x05, J4 USB_C_Receptacle_USB2.0_14P, J6 Conn_01x10, J7 Conn_01x02, J8 Conn_01x04, SW1 SW_Push, SW2 SW_Push, U1 RP2350_80QFN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

Commit message: repo cleanup
Parts:
- removed J1, J6: Conn_01x10, Connector_PinHeader_2.54mm:PinHeader_1x10_P2.54mm_Vertical_SMD_Pin1Right, symbol Connector_Generic:Conn_01x10
- removed J3: Conn_01x05, Connector_PinHeader_2.54mm:PinHeader_1x05_P2.54mm_Vertical_SMD_Pin1Right, symbol Connector_Generic:Conn_01x05
- removed J7: Conn_01x02, Connector_PinHeader_2.54mm:PinHeader_1x02_P2.54mm_Vertical_SMD_Pin1Right, symbol PCM_4ms_Connector:Conn_01x02
- added J1: Conn_01x14, Connector_PinHeader_2.54mm:PinHeader_1x14_P2.54mm_Vertical, symbol Connector_Generic:Conn_01x14
- added J5: Conn_01x12, Connector_PinHeader_2.54mm:PinHeader_1x12_P2.54mm_Vertical, symbol Connector_Generic:Conn_01x12
Connections:
- net +5V: now also J5.1 (Pin_1)
- net GND: now also J1.1 (Pin_1), J1.10 (Pin_10), J5.2 (Pin_2)
- net GPIO11: now also J5.3 (Pin_3)
- net GPIO12: now also J5.4 (Pin_4)
- net GPIO13: now also J5.5 (Pin_5)
- net GPIO14: now also J5.6 (Pin_6)
- net GPIO15: now also J5.7 (Pin_7)
- net GPIO16: now also J5.8 (Pin_8)
- net GPIO17: now also J5.9 (Pin_9)
- net GPIO18: now also J5.10 (Pin_10)
- net GPIO19: now also J5.11 (Pin_11)
- net GPIO20: now also J5.12 (Pin_12)
- net GPIO40_ADC0: now also J1.9 (Pin_9)
- net GPIO41_ADC1: now also J1.8 (Pin_8)
- net GPIO42_ADC2: now also J1.7 (Pin_7)
- net GPIO43_ADC3: now also J1.6 (Pin_6)
- net GPIO44_ADC4: now also J1.5 (Pin_5)
- net GPIO45_ADC5: now also J1.4 (Pin_4)
- net GPIO46_ADC6: now also J1.3 (Pin_3)
- net GPIO47_ADC7: now also J1.2 (Pin_2)
- net Vin_L: now also J1.14 (Pin_14)
- net Vin_R: now also J1.13 (Pin_13)
- net Vout_L: now also J1.12 (Pin_12)
- net Vout_R: now also J1.11 (Pin_11)

Commit message: change PCMxxx routing, partially route
Connections:
- net GPIO32 is gone; now on net DAC_DIN: U1.40 (GPIO32)
- net GPIO33 is gone; now on net DAC_LRCLK: U1.42 (GPIO33)
- net GPIO36 is gone; now on net ADC_SCLK: U1.45 (GPIO36)
- net GPIO37 is gone; now on net ADC_BCLK: U1.46 (GPIO37)
- net GPIO38 is gone; now on net ADC_LRCLK: U1.47 (GPIO38)
- net GPIO39 is gone; now on net ADC_DIN: U1.48 (GPIO39)
- net DAC_BCLK: now also U1.43 (GPIO34)
- net DAC_SCLK: now also U1.44 (GPIO35)
- net SCL: no longer U1.44 (GPIO35)
- net SDA: no longer U1.43 (GPIO34)
- net Vin_L: now also J1.13 (Pin_13); no longer J1.14 (Pin_14)
- net Vin_R: now also J1.14 (Pin_14); no longer J1.13 (Pin_13)
Changed lines of the file:
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@@
 	)
 	(label "ADC_SCLK"
-		(at 218.44 321.31 0)
+		(at 180.34 325.12 0)
 		(fields_autoplaced yes)
 		(effects
@@
 	)
 	(label "DAC_BCLK"
-		(at 218.44 331.47 0)
+		(at 180.34 320.04 0)
 		(fields_autoplaced yes)
 		(effects
@@
 		)
 	)
+	(label "SCL"
+		(at 189.23 307.34 0)
+		(fields_autoplaced yes)
+		(effects
+			(font
+				(size 1.27 1.27)
+			)
+			(justify left bottom)
+		)
+	)
 	(label "GPIO11"
 		(at 316.23 86.36 180)
@@
 		)
 	)
-	(label "SDA"
-		(at 180.34 320.04 0)
+	(label "ADC_DIN"
+		(at 180.34 332.74 0)
+		(fields_autoplaced yes)
+		(effects
+			(font
+				(size 1.27 1.27)
+			)
+			(justify left bottom)
+		)
+	)
+	(label "ADC_LRCLK"
+		(at 180.34 330.2 0)
 		(fields_autoplaced yes)
 		(effects
@@
 		)
 	)
-	(label "ADC_LRCLK"
-		(at 218.44 316.23 0)
-		(fields_autoplaced yes)
-		(effects
-			(font
-				(size 1.27 1.27)
-			)
-			(justify left bottom)
-		)
-	)
 	(label "GPIO40_ADC0"
 		(at 180.34 337.82 180)
@@
 		)
 	)
+	(label "GPIO35"
+		(at 180.34 322.58 180)
+		(fields_autoplaced yes)
+		(effects
+			(font
+				(size 1.27 1.27)
+			)
+			(justify right bottom)
+		)
+	)
 	(label "GPIO6"
 		(at 180.34 248.92 180)
@@
 		)
 	)
-	(label "SCL"
-		(at 180.34 322.58 0)
-		(fields_autoplaced yes)
-		(effects
-			(font
-				(size 1.27 1.27)
-			)
-			(justify left bottom)
-		)
-	)
 	(label "Vout_L"
 		(at 389.89 72.39 0)
@@
 		)
 	)
+	(label "SDA"
+		(at 189.23 304.8 0)
+		(fields_autoplaced yes)
+		(effects
+			(font
+				(size 1.27 1.27)
+			)
+			(justify left bottom)
+		)
+	)
 	(label "GPIO14"
 		(at 180.34 269.24 180)
@@
 		)
 	)
+	(label "GPIO34"
+		(at 180.34 320.04 180)
+		(fields_autoplaced yes)
+		(effects
+			(font
+				(size 1.27 1.27)
+			)
+			(justify right bottom)
+		)
+	)
+	(label "Vin_R"
+		(at 389.89 67.31 0)
+		(fields_autoplaced yes)
+		(effects
+			(font
+				(size 1.27 1.27)
+			)
+			(justify left bottom)
+		)
+	)
 	(label "GPIO14"
 		(at 316.23 93.98 180)
@@
 		)
 	)
+	(label "DAC_LRCLK"
+		(at 180.34 317.5 0)
+		(fields_autoplaced yes)
+		(effects
+			(font
+				(size 1.27 1.27)
+			)
+			(justify left bottom)
+		)
+	)
 	(label "GPIO8"
 		(at 180.34 254 180)
@@
 		)
 	)
-	(label "ADC_DIN"
-		(at 218.44 360.68 0)
-		(fields_autoplaced yes)
-		(effects
-			(font
-				(size 1.27 1.27)
-			)
-			(justify left bottom)
-		)
-	)
 	(label "XIN"
 		(at 82.55 269.24 0)
@@
 		)
 	)
-	(label "DAC_LRCLK"
-		(at 218.44 328.93 0)
-		(fields_autoplaced yes)
-		(effects
-			(font
-				(size 1.27 1.27)
-			)
-			(justify left bottom)
-		)
-	)
 	(label "GPIO12"
 		(at 316.23 88.9 180)
@@
 	)
 	(label "DAC_SCLK"
-		(at 218.44 334.01 0)
+		(at 180.34 322.58 0)
 		(fields_autoplaced yes)
 		(effects
@@
 		)
 	)
-	(label "Vin_R"
+	(label "Vin_L"
 		(at 389.89 69.85 0)
 		(fields_autoplaced yes)
@@
 	)
 	(label "ADC_BCLK"
-		(at 218.44 318.77 0)
+		(at 180.34 327.66 0)
 		(fields_autoplaced yes)
 		(effects
@@
 	)
 	(label "DAC_DIN"
-		(at 218.44 326.39 0)
-		(fields_autoplaced yes)
-		(effects
-			(font
-				(size 1.27 1.27)
-			)
-			(justify left bottom)
-		)
-	)
-	(label "Vin_L"
-		(at 389.89 67.31 0)
-		(fields_autoplaced yes)
-		(effects
+		(at 180.34 314.96 0)
+		(fields_autoplaced yes)
+		(effects
